File: hardware/turbocan.kicad_sch (KiCad schematic)
At the start: 88 parts, among them J1 USB_C_Receptacle_USB2.0, J10 CAN_PORT, J11 FAN0, J12 FAN1, J13 HEAT, J14 PROBE, J2 STEPPER, J5 DEBUG, J7 ENDSTOPX, J8 ENDSTOPY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

Commit message: Updated schematic with generic IO, removed ADXL.
Parts:
- removed R12, R13: 1k, Resistor_SMD:R_0402_1005Metric, symbol archive:Device_R_Small
- removed U9: ADXL345BCCZ, digikey-footprints:LGA-14_3x5mm_RevA, symbol archive:dk_Motion-Sensors-Accelerometers_ADXL345BCCZ
- added C?: 100nF, Capacitor_SMD:C_0402_1005Metric, symbol archive:Device_C_Small
- added J15: SPI, Connector_JST:JST_XH_B6B-XH-A_1x06_P2.50mm_Vertical, symbol Connector:Conn_01x06_Male
- added J?: IO_PB10, Connector_JST:JST_XH_B3B-XH-A_1x03_P2.50mm_Vertical, symbol archive:Connector_Conn_01x03_Male
- added R?: 10k, Resistor_SMD:R_0402_1005Metric, symbol archive:Device_R_Small
- added R?: 1K, Resistor_THT:R_Axial_DIN0204_L3.6mm_D1.6mm_P2.54mm_Vertical, symbol Device:R
- J1: now left out of the parts list
- J7: value ENDSTOPX -> IO_PB6
- J8: value ENDSTOPY -> IO_PB7
Connections:
- net ENDSTOPX is gone; now on net IO1: U8.42 (PB6)
- net ENDSTOPY is gone; now on net IO2: U8.43 (PB7)
- net +3V3: now also R?.1
- net +5V: now also J15.2 (Pin_2), J?.1 (Pin_1)
- net A_CS: now also J15.3 (Pin_3)
- net A_MISO: now also J15.5 (Pin_5)
- net A_MOSI: now also J15.4 (Pin_4)
- net A_SCK: now also J15.6 (Pin_6)
- net GND: now also J15.1 (Pin_1), J?.2 (Pin_2)
- net TH0: now also R?.2
- net VDDA: now also R?.1
- net IO3: now reaches U8.21 (PB10)
- net IO3: now also C?.1, J?.3 (Pin_3), R?.2
- net IO1: now reaches C10.1, J7.3 (Pin_3), R7.2
- net IO2: now reaches C11.1, J8.3 (Pin_3), R8.2
- net CANH: no longer names the net of J10.2 (Pin_2), R26.1, U3.7 (CANH)
- net CANL: no longer names the net of J10.3 (Pin_3), R26.2, U3.6 (CANL)
- no-connect marks 14 -> 9
Other:
- note added: "INPUT/OUTPUT"
- note added: "POWER INPUT"
- note removed: "X/Y/Z ENDSTOPS"
- moved on the sheet: C1, C10, C11, C12, C13, C14, C15, C16, C17, C18, C19, C2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

Commit message: First Test
Parts:
- removed R1, R2: 5.1k, Resistor_SMD:R_0402_1005Metric, symbol archive:Device_R_Small
- removed R?: 1K, Resistor_THT:R_Axial_DIN0204_L3.6mm_D1.6mm_P2.54mm_Vertical, symbol Device:R
- J1: value USB_C_Receptacle_USB2.0 -> USB_B_Micro_Receptacle_USB2.0; footprint Connector_USB:USB_C_Receptacle_HRO_TYPE-C-31-M-12 -> Connector_USB:USB_Micro-B_Amphenol_10118194_Horizontal; symbol archive:Connector_USB_C_Receptacle_USB2.0 -> Connector:USB_B_Micro; now in the parts list
- gave numbers to parts that had none: 3
Connections:
- net GND: now also J1.5 (GND), J1.6 (Shield); no longer J1.A1 (GND), J1.A12 (GND), J1.B1 (GND), J1.B12 (GND), J1.S1 (SHIELD)
- net USBDM: now also J1.2 (D-); no longer J1.A7 (D-), J1.B7 (D-)
- net USBDP: now also J1.3 (D+); no longer J1.A6 (D+), J1.B6 (D+)
- new net: D1.2 (A), J1.1 (VBUS)
- no-connect marks 9 -> 8
Other:
- note added: "USB-B Micro"
- note removed: "USB-C"
- moved on the sheet: D1

Commit message: Before DRC
Parts:
- removed H2, H3: MountingHole, MountingHole:MountingHole_3.2mm_M3_DIN965_Pad, symbol archive:Mechanical_MountingHole
- removed J5: DEBUG, Connector_PinHeader_2.54mm:PinHeader_2x03_P2.54mm_Vertical, symbol archive:Connector_Generic_Conn_02x03_Odd_Even
- added JP1: SolderJumper_2_Open, Jumper:SolderJumper-2_P1.3mm_Open_TrianglePad1.0x1.5mm, symbol Jumper:SolderJumper_2_Open
- J15: footprint Connector_JST:JST_XH_B6B-XH-A_1x06_P2.50mm_Vertical -> Connector_PinHeader_2.54mm:PinHeader_2x03_P2.54mm_Vertical; symbol Connector:Conn_01x06_Male -> Connector_Generic:Conn_02x03_Top_Bottom
- R23: value 1k -> 10k
Connections:
- net +24V: now also D5.2 (A)
- net +3V3: now also JP1.1 (A); no longer D6.2 (A), R2.1, R7.1, R8.1
- net +5V: now also D6.2 (A), J15.5 (Pin_5), R2.1, R7.1, R8.1; no longer J15.2 (Pin_2)
- net A_CS: now also J15.6 (Pin_6); no longer J15.3 (Pin_3)
- net A_MISO: now also J15.4 (Pin_4); no longer J15.5 (Pin_5)
- net A_MOSI: now also J15.2 (Pin_2); no longer J15.4 (Pin_4)
- net A_SCK: now also J15.3 (Pin_3); no longer J15.6 (Pin_6)
- net BOOT0: now also JP1.2 (B)
- net GND: now also C24.2; no longer R23.2
- net IO3: now also U8.11 (PA1); no longer U8.21 (PB10)
- net PROBEZ: now also U8.38 (PA15); no longer U8.22 (PB11)
- net at J13.1 (Pin_1), U7.3 (D): now also R23.2
- removed net LED: D5.2 (A), U8.11 (PA1)
- net USBDM renamed USBDN
- no-connect marks 8 -> 9
Other:
- note added: "SPI BREAKOUT"
- moved on the sheet: D5, R16, R19, R23, U7

Commit message: First Manufacturing Upload
Connections:
- net GND: no longer J1.6 (Shield)
- no-connect marks 9 -> 10
Changed lines of the file:
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@@
   (junction (at 176.53 256.54) (diameter 0) (color 0 0 0 0)
-  )
-  (junction (at 77.47 60.96) (diameter 0) (color 0 0 0 0)
   )
   (junction (at 273.05 57.15) (diameter 0) (color 0 0 0 0)
@@
   (no_connect (at 356.87 60.96))
   (no_connect (at 356.87 66.04))
+  (no_connect (at 77.47 58.42))
   (no_connect (at 48.26 267.97))
   (no_connect (at 356.87 96.52))
@@
     (stroke (width 0) (type default) (color 0 0 0 0))
   )
-  (wire (pts (xy 80.01 60.96) (xy 77.47 60.96))
-    (stroke (width 0) (type default) (color 0 0 0 0))
-  )
   (wire (pts (xy 229.87 261.62) (xy 229.87 267.97))
     (stroke (width 0) (type default) (color 0 0 0 0))
@@
     (stroke (width 0) (type default) (color 0 0 0 0))
   )
-  (wire (pts (xy 77.47 60.96) (xy 77.47 62.23))
-    (stroke (width 0) (type default) (color 0 0 0 0))
-  )
   (wire (pts (xy 73.66 269.24) (xy 93.98 269.24))
     (stroke (width 0) (type default) (color 0 0 0 0))
@@
   )
   (wire (pts (xy 90.17 266.7) (xy 93.98 266.7))
-    (stroke (width 0) (type default) (color 0 0 0 0))
-  )
-  (wire (pts (xy 77.47 58.42) (xy 77.47 60.96))
     (stroke (width 0) (type default) (color 0 0 0 0))
   )
@@
     (pin "2")
   )
-  (symbol (lib_id "archive:power_GND") (at 77.47 62.23 0) (unit 1)
-    (in_bom yes) (on_board yes)
-    (property "Reference" "#PWR01" (id 0) (at 77.47 68.58 0)
-      (effects (font (size 1.27 1.27)) hide)
-    )
-    (property "Value" "GND" (id 1) (at 77.597 66.6242 0))
-    (property "Footprint" "" (id 2) (at 77.47 62.23 0)
-      (effects (font (size 1.27 1.27)) hide)
-    )
-    (property "Datasheet" "" (id 3) (at 77.47 62.23 0)
-      (effects (font (size 1.27 1.27)) hide)
-    )
+  (symbol (lib_id "archive:power_GND") (at 80.01 60.96 0) (unit 1)
+    (in_bom yes) (on_board yes)
+    (property "Reference" "#PWR01" (id 0) (at 80.01 67.31 0)
+      (effects (font (size 1.27 1.27)) hide)
+    )
+    (property "Value" "GND" (id 1) (at 80.137 65.3542 0))
+    (property "Footprint" "" (id 2) (at 80.01 60.96 0)
+      (effects (font (size 1.27 1.27)) hide)
+    )
+    (property "Datasheet" "" (id 3) (at 80.01 60.96 0)
+      (effects (font (size 1.27 1.27)) hide)
+    )
